File: Stepper Motor Driver.sch (KiCad schematic (older format))
At the start: 5 parts, among them T1 L298, T2 L298, T3 L298, T4 L298, T5 L298

Commit message: Started hierarchical schematic
Parts:
- removed T1, T2, T3, T4, T5: L298, Multiwatt15, symbol L298
Connections:
- net labels removed: +5V, GND, T1_Enable_A, T1_Enable_B, T1_Input_2, T1_Input_3, T1_Input_4, T1_Output_1, T1_Output_2, T1_Output_3, T1_Output_4, T2_Enable_A, T2_Enable_B, T2_Input_1, T2_Input_2, T2_Input_3, T2_Input_4, T2_Output_1, T2_Output_2, T2_Output_3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
- wire segments 50 -> 0
