File: Top.sch (KiCad schematic (older format))
At the start: 0 parts

Commit message: New schematics: Top and Controller
Changed lines of the file:
@@
 LIBS:contrib
 LIBS:valves
-LIBS:Stepper Motor Driver-cache
+LIBS:Driver-cache
 EELAYER 25 0
 EELAYER END
 $Descr A4 11693 8268
 encoding utf-8
-Sheet 1 2
+Sheet 1 3
 Title ""
 Date ""
@@
 $EndDescr
 $Sheet
-S 7050 3100 1300 1300
-U 5A1C80E3
+S 2300 2800 1600 1500
+U 5A1D9334
+F0 "Controller" 60
+F1 "Controller.sch" 60
+$EndSheet
+$Sheet
+S 4550 2800 1650 1750
+U 5A1D933F
 F0 "Transistors" 60
 F1 "Transistors.sch" 60
+F2 "T1_Enable_A" I L 4550 3000 60
+F3 "T1_Input_2" I L 4550 3100 60
+F4 "T1_Input_3" I L 4550 3350 60
+F5 "T1_Enable_B" I L 4550 3450 60
+F6 "T1_Input_4" I L 4550 3550 60
+F7 "T1_Output_1" I L 4550 3750 60
+F8 "T1_Output_2" I L 4550 3950 60
+F9 "T1_Output_3" I R 6200 3200 60
 $EndSheet
-Text HLabel 8350 3250 0    60   Input ~ 0
-T1_Input_1
 $EndSCHEMATC
