File: L298.sch (KiCad schematic (older format))
At the start: 3 parts

Commit message: Added Multiwatt15 footprint to L298
Parts:
- T: footprint Multiwatt15 -> TO_SOT_Packages_THT:Multiwatt-15_Vertical_StaggeredType1
Changed lines of the file:
@@
 EESchema Schematic File Version 2
+LIBS:L298
 LIBS:power
 LIBS:device
@@
 LIBS:contrib
 LIBS:valves
+LIBS:Top-cache
 EELAYER 25 0
 EELAYER END
 $Descr A4 11693 8268
 encoding utf-8
-Sheet 4 4
+Sheet 8 8
 Title ""
 Date ""
@@
 F 0 "T" H 6700 3200 60  0000 C CNN
 F 1 "L298" H 5800 4600 60  0000 C CNN
-F 2 "Multiwatt15" H 5500 3000 60  0001 C CNN
+F 2 "TO_SOT_Packages_THT:Multiwatt-15_Vertical_StaggeredType1" H 5500 3000 60  0001 C CNN
 F 3 "" H 6300 3900 60  0001 C CNN
 	1    6300 3900

Commit message: Schematic annotated successfully
Parts:
- renumbered T to T1, T_C1 to T_C1_1, T_C2 to T_C2_1
Changed lines of the file:
@@
 $Descr A4 11693 8268
 encoding utf-8
-Sheet 8 8
+Sheet 4 8
 Title ""
 Date ""
@@
 $EndDescr
 $Comp
-L L298 T
+L L298 T1
 U 1 1 5A2054BE
 P 6300 3900
-F 0 "T" H 6700 3200 60  0000 C CNN
+AR Path="/5A23F11B/5A20538E/5A2054BE" Ref="T1"  Part="1"
+AR Path="/5A23F11B/5A209EE3/5A2054BE" Ref="T2"  Part="1"
+AR Path="/5A23F11B/5A20B0FB/5A2054BE" Ref="T3"  Part="1"
+AR Path="/5A23F11B/5A20C9FB/5A2054BE" Ref="T4"  Part="1"
+AR Path="/5A23F11B/5A20D3A3/5A2054BE" Ref="T5"  Part="1"
+F 0 "T1" H 6700 3200 60  0000 C CNN
 F 1 "L298" H 5800 4600 60  0000 C CNN
 F 2 "TO_SOT_Packages_THT:Multiwatt-15_Vertical_StaggeredType1" H 5500 3000 60  0001 C CNN
@@
 Input_4
 $Comp
-L GNDD #PWR?
+L GNDD #PWR4
 U 1 1 5A206647
 P 6100 4700
-F 0 "#PWR?" H 6100 4450 50  0001 C CNN
+AR Path="/5A23F11B/5A20538E/5A206647" Ref="#PWR4"  Part="1"
+AR Path="/5A23F11B/5A209EE3/5A206647" Ref="#PWR12"  Part="1"
+AR Path="/5A23F11B/5A20B0FB/5A206647" Ref="#PWR20"  Part="1"
+AR Path="/5A23F11B/5A20C9FB/5A206647" Ref="#PWR28"  Part="1"
+AR Path="/5A23F11B/5A20D3A3/5A206647" Ref="#PWR36"  Part="1"
+F 0 "#PWR4" H 6100 4450 50  0001 C CNN
 F 1 "GNDD" H 6100 4575 50  0000 C CNN
 F 2 "" H 6100 4700 50  0001 C CNN
@@
 $EndComp
 $Comp
-L VDD #PWR?
+L VDD #PWR5
 U 1 1 5A206674
 P 6400 3100
-F 0 "#PWR?" H 6400 2950 50  0001 C CNN
+AR Path="/5A23F11B/5A20538E/5A206674" Ref="#PWR5"  Part="1"
+AR Path="/5A23F11B/5A209EE3/5A206674" Ref="#PWR13"  Part="1"
+AR Path="/5A23F11B/5A20B0FB/5A206674" Ref="#PWR21"  Part="1"
+AR Path="/5A23F11B/5A20C9FB/5A206674" Ref="#PWR29"  Part="1"
+AR Path="/5A23F11B/5A20D3A3/5A206674" Ref="#PWR37"  Part="1"
+F 0 "#PWR5" H 6400 2950 50  0001 C CNN
 F 1 "VDD" H 6400 3250 50  0000 C CNN
 F 2 "" H 6400 3100 50  0001 C CNN
@@
 	6400 4700 6300 4700
 $Comp
-L +5V #PWR?
+L +5V #PWR3
 U 1 1 5A20668C
 P 6100 3100
-F 0 "#PWR?" H 6100 2950 50  0001 C CNN
+AR Path="/5A23F11B/5A20538E/5A20668C" Ref="#PWR3"  Part="1"
+AR Path="/5A23F11B/5A209EE3/5A20668C" Ref="#PWR11"  Part="1"
+AR Path="/5A23F11B/5A20B0FB/5A20668C" Ref="#PWR19"  Part="1"
+AR Path="/5A23F11B/5A20C9FB/5A20668C" Ref="#PWR27"  Part="1"
+AR Path="/5A23F11B/5A20D3A3/5A20668C" Ref="#PWR35"  Part="1"
+F 0 "#PWR3" H 6100 2950 50  0001 C CNN
 F 1 "+5V" H 6100 3240 50  0000 C CNN
 F 2 "" H 6100 3100 50  0001 C CNN
@@
 Output_4
 $Comp
-L +5V #PWR?
+L +5V #PWR1
 U 1 1 5A20673C
 P 5250 2950
-F 0 "#PWR?" H 5250 2800 50  0001 C CNN
+AR Path="/5A23F11B/5A20538E/5A20673C" Ref="#PWR1"  Part="1"
+AR Path="/5A23F11B/5A209EE3/5A20673C" Ref="#PWR9"  Part="1"
+AR Path="/5A23F11B/5A20B0FB/5A20673C" Ref="#PWR17"  Part="1"
+AR Path="/5A23F11B/5A20C9FB/5A20673C" Ref="#PWR25"  Part="1"
+AR Path="/5A23F11B/5A20D3A3/5A20673C" Ref="#PWR33"  Part="1"
+F 0 "#PWR1" H 5250 2800 50  0001 C CNN
 F 1 "+5V" H 5250 3090 50  0000 C CNN
 F 2 "" H 5250 2950 50  0001 C CNN
@@
 $EndComp
 $Comp
-L GNDD #PWR?
+L GNDD #PWR2
 U 1 1 5A206752
 P 5250 3150
-F 0 "#PWR?" H 5250 2900 50  0001 C CNN
+AR Path="/5A23F11B/5A20538E/5A206752" Ref="#PWR2"  Part="1"
+AR Path="/5A23F11B/5A209EE3/5A206752" Ref="#PWR10"  Part="1"
+AR Path="/5A23F11B/5A20B0FB/5A206752" Ref="#PWR18"  Part="1"
+AR Path="/5A23F11B/5A20C9FB/5A206752" Ref="#PWR26"  Part="1"
+AR Path="/5A23F11B/5A20D3A3/5A206752" Ref="#PWR34"  Part="1"
+F 0 "#PWR2" H 5250 2900 50  0001 C CNN
 F 1 "GNDD" H 5250 3025 50  0000 C CNN
 F 2 "" H 5250 3150 50  0001 C CNN
@@
 $EndComp
 $Comp
-L VDD #PWR?
+L VDD #PWR7
 U 1 1 5A20677E
 P 7200 2950
-F 0 "#PWR?" H 7200 2800 50  0001 C CNN
+AR Path="/5A23F11B/5A20538E/5A20677E" Ref="#PWR7"  Part="1"
+AR Path="/5A23F11B/5A209EE3/5A20677E" Ref="#PWR15"  Part="1"
+AR Path="/5A23F11B/5A20B0FB/5A20677E" Ref="#PWR23"  Part="1"
+AR Path="/5A23F11B/5A20C9FB/5A20677E" Ref="#PWR31"  Part="1"
+AR Path="/5A23F11B/5A20D3A3/5A20677E" Ref="#PWR39"  Part="1"
+F 0 "#PWR7" H 7200 2800 50  0001 C CNN
 F 1 "VDD" H 7200 3100 50  0000 C CNN
 F 2 "" H 7200 2950 50  0001 C CNN
@@
 $EndComp
 $Comp
-L VSS #PWR?
+L VSS #PWR8
 U 1 1 5A2067B4
 P 7200 3150
-F 0 "#PWR?" H 7200 3000 50  0001 C CNN
+AR Path="/5A23F11B/5A20538E/5A2067B4" Ref="#PWR8"  Part="1"
+AR Path="/5A23F11B/5A209EE3/5A2067B4" Ref="#PWR16"  Part="1"
+AR Path="/5A23F11B/5A20B0FB/5A2067B4" Ref="#PWR24"  Part="1"
+AR Path="/5A23F11B/5A20C9FB/5A2067B4" Ref="#PWR32"  Part="1"
+AR Path="/5A23F11B/5A20D3A3/5A2067B4" Ref="#PWR40"  Part="1"
+F 0 "#PWR8" H 7200 3000 50  0001 C CNN
 F 1 "VSS" H 7200 3300 50  0000 C CNN
 F 2 "" H 7200 3150 50  0001 C CNN
@@
 $EndComp
 $Comp
-L C_Small T_C1
+L C_Small T_C1_1
 U 1 1 5A2067CA
 P 5250 3050
-F 0 "T_C1" H 5260 3120 50  0000 L CNN
+AR Path="/5A23F11B/5A20538E/5A2067CA" Ref="T_C1_1"  Part="1"
+AR Path="/5A23F11B/5A209EE3/5A2067CA" Ref="T_C1_2"  Part="1"
+AR Path="/5A23F11B/5A20B0FB/5A2067CA" Ref="T_C1_3"  Part="1"
+AR Path="/5A23F11B/5A20C9FB/5A2067CA" Ref="T_C1_4"  Part="1"
+AR Path="/5A23F11B/5A20D3A3/5A2067CA" Ref="T_C1_5"  Part="1"
+F 0 "T_C1_1" H 5260 3120 50  0000 L CNN
 F 1 "100nF" H 5260 2970 50  0000 L CNN
 F 2 "" H 5250 3050 50  0001 C CNN
@@
 $EndComp
 $Comp
-L C_Small T_C2
+L C_Small T_C2_1
 U 1 1 5A2067FF
 P 7200 3050
-F 0 "T_C2" H 7210 3120 50  0000 L CNN
+AR Path="/5A23F11B/5A20538E/5A2067FF" Ref="T_C2_1"  Part="1"
+AR Path="/5A23F11B/5A209EE3/5A2067FF" Ref="T_C2_2"  Part="1"
+AR Path="/5A23F11B/5A20B0FB/5A2067FF" Ref="T_C2_3"  Part="1"
+AR Path="/5A23F11B/5A20C9FB/5A2067FF" Ref="T_C2_4"  Part="1"
+AR Path="/5A23F11B/5A20D3A3/5A2067FF" Ref="T_C2_5"  Part="1"
+F 0 "T_C2_1" H 7210 3120 50  0000 L CNN
 F 1 "100nF" H 7210 2970 50  0000 L CNN
 F 2 "" H 7200 3050 50  0001 C CNN
@@
 $EndComp
 $Comp
-L VSS #PWR?
+L VSS #PWR6
 U 1 1 5A206BC4
 P 6400 4700
-F 0 "#PWR?" H 6400 4550 50  0001 C CNN
+AR Path="/5A23F11B/5A20538E/5A206BC4" Ref="#PWR6"  Part="1"
+AR Path="/5A23F11B/5A209EE3/5A206BC4" Ref="#PWR14"  Part="1"
+AR Path="/5A23F11B/5A20B0FB/5A206BC4" Ref="#PWR22"  Part="1"
+AR Path="/5A23F11B/5A20C9FB/5A206BC4" Ref="#PWR30"  Part="1"
+AR Path="/5A23F11B/5A20D3A3/5A206BC4" Ref="#PWR38"  Part="1"
+F 0 "#PWR6" H 6400 4550 50  0001 C CNN
 F 1 "VSS" H 6400 4850 50  0000 C CNN
 F 2 "" H 6400 4700 50  0001 C CNN
