File: L298.sch (KiCad schematic (older format))
At the start: 3 parts, among them T1 L298

Commit message: Added and connected sixth L298N symbol
Changed lines of the file:
@@
 $Descr A4 11693 8268
 encoding utf-8
-Sheet 7 10
+Sheet 6 11
 Title ""
 Date ""
@@
 AR Path="/5A23F11B/5A20C9FB/5A2054BE" Ref="T4"  Part="1"
 AR Path="/5A23F11B/5A20D3A3/5A2054BE" Ref="T5"  Part="1"
-F 0 "T4" H 6700 3200 60  0000 C CNN
+AR Path="/5A23F11B/5A274D45/5A2054BE" Ref="T6"  Part="1"
+F 0 "T1" H 6700 3200 60  0000 C CNN
 F 1 "L298" H 5800 4600 60  0000 C CNN
 F 2 "TO_SOT_Packages_THT:Multiwatt-15_Vertical_StaggeredType1" H 5500 3000 60  0001 C CNN
@@
 AR Path="/5A23F11B/5A20C9FB/5A206647" Ref="#PWR28"  Part="1"
 AR Path="/5A23F11B/5A20D3A3/5A206647" Ref="#PWR36"  Part="1"
-F 0 "#PWR28" H 6100 4450 50  0001 C CNN
+AR Path="/5A23F11B/5A274D45/5A206647" Ref="#PWR44"  Part="1"
+F 0 "#PWR4" H 6100 4450 50  0001 C CNN
 F 1 "GNDD" H 6100 4575 50  0000 C CNN
 F 2 "" H 6100 4700 50  0001 C CNN
@@
 AR Path="/5A23F11B/5A20C9FB/5A206674" Ref="#PWR29"  Part="1"
 AR Path="/5A23F11B/5A20D3A3/5A206674" Ref="#PWR37"  Part="1"
-F 0 "#PWR29" H 6400 2950 50  0001 C CNN
+AR Path="/5A23F11B/5A274D45/5A206674" Ref="#PWR45"  Part="1"
+F 0 "#PWR5" H 6400 2950 50  0001 C CNN
 F 1 "VDD" H 6400 3250 50  0000 C CNN
 F 2 "" H 6400 3100 50  0001 C CNN
@@
 AR Path="/5A23F11B/5A20C9FB/5A20668C" Ref="#PWR27"  Part="1"
 AR Path="/5A23F11B/5A20D3A3/5A20668C" Ref="#PWR35"  Part="1"
-F 0 "#PWR27" H 6100 2950 50  0001 C CNN
+AR Path="/5A23F11B/5A274D45/5A20668C" Ref="#PWR43"  Part="1"
+F 0 "#PWR3" H 6100 2950 50  0001 C CNN
 F 1 "+5V" H 6100 3240 50  0000 C CNN
 F 2 "" H 6100 3100 50  0001 C CNN
@@
 AR Path="/5A23F11B/5A20C9FB/5A20673C" Ref="#PWR25"  Part="1"
 AR Path="/5A23F11B/5A20D3A3/5A20673C" Ref="#PWR33"  Part="1"
-F 0 "#PWR25" H 5250 2800 50  0001 C CNN
+AR Path="/5A23F11B/5A274D45/5A20673C" Ref="#PWR41"  Part="1"
+F 0 "#PWR1" H 5250 2800 50  0001 C CNN
 F 1 "+5V" H 5250 3090 50  0000 C CNN
 F 2 "" H 5250 2950 50  0001 C CNN
@@
 AR Path="/5A23F11B/5A20C9FB/5A206752" Ref="#PWR26"  Part="1"
 AR Path="/5A23F11B/5A20D3A3/5A206752" Ref="#PWR34"  Part="1"
-F 0 "#PWR26" H 5250 2900 50  0001 C CNN
+AR Path="/5A23F11B/5A274D45/5A206752" Ref="#PWR42"  Part="1"
+F 0 "#PWR2" H 5250 2900 50  0001 C CNN
 F 1 "GNDD" H 5250 3025 50  0000 C CNN
 F 2 "" H 5250 3150 50  0001 C CNN
@@
 AR Path="/5A23F11B/5A20C9FB/5A20677E" Ref="#PWR31"  Part="1"
 AR Path="/5A23F11B/5A20D3A3/5A20677E" Ref="#PWR39"  Part="1"
-F 0 "#PWR31" H 7200 2800 50  0001 C CNN
+AR Path="/5A23F11B/5A274D45/5A20677E" Ref="#PWR47"  Part="1"
+F 0 "#PWR7" H 7200 2800 50  0001 C CNN
 F 1 "VDD" H 7200 3100 50  0000 C CNN
 F 2 "" H 7200 2950 50  0001 C CNN
@@
 AR Path="/5A23F11B/5A20C9FB/5A2067B4" Ref="#PWR32"  Part="1"
 AR Path="/5A23F11B/5A20D3A3/5A2067B4" Ref="#PWR40"  Part="1"
-F 0 "#PWR32" H 7200 3000 50  0001 C CNN
+AR Path="/5A23F11B/5A274D45/5A2067B4" Ref="#PWR48"  Part="1"
+F 0 "#PWR8" H 7200 3000 50  0001 C CNN
 F 1 "VSS" H 7200 3300 50  0000 C CNN
 F 2 "" H 7200 3150 50  0001 C CNN
@@
 AR Path="/5A23F11B/5A20C9FB/5A2067CA" Ref="T_C1_4"  Part="1"
 AR Path="/5A23F11B/5A20D3A3/5A2067CA" Ref="T_C1_5"  Part="1"
-F 0 "T_C1_4" H 5260 3120 50  0000 L CNN
+AR Path="/5A23F11B/5A274D45/5A2067CA" Ref="T_C1_6"  Part="1"
+F 0 "T_C1_1" H 5260 3120 50  0000 L CNN
 F 1 "100nF" H 5260 2970 50  0000 L CNN
 F 2 "" H 5250 3050 50  0001 C CNN
@@
 AR Path="/5A23F11B/5A20C9FB/5A2067FF" Ref="T_C2_4"  Part="1"
 AR Path="/5A23F11B/5A20D3A3/5A2067FF" Ref="T_C2_5"  Part="1"
-F 0 "T_C2_4" H 7210 3120 50  0000 L CNN
+AR Path="/5A23F11B/5A274D45/5A2067FF" Ref="T_C2_6"  Part="1"
+F 0 "T_C2_1" H 7210 3120 50  0000 L CNN
 F 1 "100nF" H 7210 2970 50  0000 L CNN
 F 2 "" H 7200 3050 50  0001 C CNN
@@
 AR Path="/5A23F11B/5A20C9FB/5A206BC4" Ref="#PWR30"  Part="1"
 AR Path="/5A23F11B/5A20D3A3/5A206BC4" Ref="#PWR38"  Part="1"
-F 0 "#PWR30" H 6400 4550 50  0001 C CNN
+AR Path="/5A23F11B/5A274D45/5A206BC4" Ref="#PWR46"  Part="1"
+F 0 "#PWR6" H 6400 4550 50  0001 C CNN
 F 1 "VSS" H 6400 4850 50  0000 C CNN
 F 2 "" H 6400 4700 50  0001 C CNN
