File: Chopper.sch (KiCad schematic (older format))
At the start: 0 parts

Commit message: Moved OpAmp to Chopper.sch
Parts:
- added Q?: Q_NMOS_GDS, symbol Q_NMOS_GDS
- added R? (x3): R_Small, symbol R_Small
- added U? (x2): LM358, symbol LM358
Connections:
- net labels added: +5V, GNDPWR, current_desired, current_measured, current_scaled
- wire segments 0 -> 6
Changed lines of the file:
@@
 Comment4 ""
 $EndDescr
+$Comp
+L Q_NMOS_GDS Q?
+U 1 1 5A2B4511
+P 7650 3800
+AR Path="/5A2AF2A6/5A2B8CFF/5A2B4511" Ref="Q?"  Part="1"
+AR Path="/5A2AF2A6/5A2B8A78/5A2B4511" Ref="Q?"  Part="1"
+F 0 "Q?" H 7850 3850 50  0000 L CNN
+F 1 "Q_NMOS_GDS" H 7850 3750 50  0000 L CNN
+F 2 "" H 7850 3900 50  0001 C CNN
+F 3 "" H 7650 3800 50  0001 C CNN
+	1    7650 3800
+	1    0    0    -1
+$EndComp
+$Comp
+L LM358 U?
+U 1 1 5A2B487D
+P 6650 2000
+AR Path="/5A2AF2A6/5A2B8CFF/5A2B487D" Ref="U?"  Part="1"
+AR Path="/5A2AF2A6/5A2B8A78/5A2B487D" Ref="U?"  Part="1"
+F 0 "U?" H 6650 2200 50  0000 L CNN
+F 1 "LM358" H 6650 1800 50  0000 L CNN
+F 2 "" H 6650 2000 50  0001 C CNN
+F 3 "" H 6650 2000 50  0001 C CNN
+	1    6650 2000
+	1    0    0    -1
+$EndComp
+$Comp
+L LM358 U?
+U 2 1 5A2B48DE
+P 6600 3800
+AR Path="/5A2AF2A6/5A2B8CFF/5A2B48DE" Ref="U?"  Part="2"
+AR Path="/5A2AF2A6/5A2B8A78/5A2B48DE" Ref="U?"  Part="2"
+F 0 "U?" H 6600 4000 50  0000 L CNN
+F 1 "LM358" H 6600 3600 50  0000 L CNN
+F 2 "" H 6600 3800 50  0001 C CNN
+F 3 "" H 6600 3800 50  0001 C CNN
+	2    6600 3800
+	1    0    0    -1
+$EndComp
+$Comp
+L +5V #PWR?
+U 1 1 5A2B4ABD
+P 6500 3500
+AR Path="/5A2AF2A6/5A2B8CFF/5A2B4ABD" Ref="#PWR?"  Part="1"
+AR Path="/5A2AF2A6/5A2B8A78/5A2B4ABD" Ref="#PWR?"  Part="1"
+F 0 "#PWR?" H 6500 3350 50  0001 C CNN
+F 1 "+5V" H 6500 3640 50  0000 C CNN
+F 2 "" H 6500 3500 50  0001 C CNN
+F 3 "" H 6500 3500 50  0001 C CNN
+	1    6500 3500
+	1    0    0    -1
+$EndComp
+$Comp
+L +5V #PWR?
+U 1 1 5A2B4B1F
+P 6550 1700
+AR Path="/5A2AF2A6/5A2B8CFF/5A2B4B1F" Ref="#PWR?"  Part="1"
+AR Path="/5A2AF2A6/5A2B8A78/5A2B4B1F" Ref="#PWR?"  Part="1"
+F 0 "#PWR?" H 6550 1550 50  0001 C CNN
+F 1 "+5V" H 6550 1840 50  0000 C CNN
+F 2 "" H 6550 1700 50  0001 C CNN
+F 3 "" H 6550 1700 50  0001 C CNN
+	1    6550 1700
+	1    0    0    -1
+$EndComp
+$Comp
+L GNDPWR #PWR?
+U 1 1 5A2B4F34
+P 6550 2300
+AR Path="/5A2AF2A6/5A2B8CFF/5A2B4F34" Ref="#PWR?"  Part="1"
+AR Path="/5A2AF2A6/5A2B8A78/5A2B4F34" Ref="#PWR?"  Part="1"
+F 0 "#PWR?" H 6550 2100 50  0001 C CNN
+F 1 "GNDPWR" H 6550 2150 50  0000 C CNN
+F 2 "" H 6550 2250 50  0001 C CNN
+F 3 "" H 6550 2250 50  0001 C CNN
+	1    6550 2300
+	1    0    0    -1
+$EndComp
+$Comp
+L GNDPWR #PWR?
+U 1 1 5A2B4F6B
+P 6500 4100
+AR Path="/5A2AF2A6/5A2B8CFF/5A2B4F6B" Ref="#PWR?"  Part="1"
+AR Path="/5A2AF2A6/5A2B8A78/5A2B4F6B" Ref="#PWR?"  Part="1"
+F 0 "#PWR?" H 6500 3900 50  0001 C CNN
+F 1 "GNDPWR" H 6500 3950 50  0000 C CNN
+F 2 "" H 6500 4050 50  0001 C CNN
+F 3 "" H 6500 4050 50  0001 C CNN
+	1    6500 4100
+	1    0    0    -1
+$EndComp
+$Comp
+L R_Small R?
+U 1 1 5A2B531C
+P 7200 3800
+AR Path="/5A2AF2A6/5A2B8CFF/5A2B531C" Ref="R?"  Part="1"
+AR Path="/5A2AF2A6/5A2B8A78/5A2B531C" Ref="R?"  Part="1"
+F 0 "R?" V 7100 3750 50  0000 L CNN
+F 1 "R_Small" V 7300 3700 50  0000 L CNN
+F 2 "" H 7200 3800 50  0001 C CNN
+F 3 "" H 7200 3800 50  0001 C CNN
+	1    7200 3800
+	0    1    1    0
+$EndComp
+Wire Wire Line
+	7300 3800 7450 3800
+Wire Wire Line
+	7100 3800 6900 3800
+$Comp
+L GNDPWR #PWR?
+U 1 1 5A2B5A80
+P 7750 4000
+AR Path="/5A2AF2A6/5A2B8CFF/5A2B5A80" Ref="#PWR?"  Part="1"
+AR Path="/5A2AF2A6/5A2B8A78/5A2B5A80" Ref="#PWR?"  Part="1"
+F 0 "#PWR?" H 7750 3800 50  0001 C CNN
+F 1 "GNDPWR" H 7750 3850 50  0000 C CNN
+F 2 "" H 7750 3950 50  0001 C CNN
+F 3 "" H 7750 3950 50  0001 C CNN
+	1    7750 4000
+	1    0    0    -1
+$EndComp
+Wire Wire Line
+	6300 3900 5900 3900
+Wire Wire Line
+	6300 3700 5900 3700
+Text GLabel 5900 3900 0    60   Input ~ 0
+current_scaled
+Text GLabel 5900 3700 0    60   Input ~ 0
+current_desired
+Text GLabel 8000 2000 0    60   Output ~ 0
+current_scaled
+Wire Wire Line
+	7300 2000 6950 2000
+Wire Wire Line
+	6350 1900 5950 1900
+Text GLabel 5950 1900 0    60   Input ~ 0
+current_measured
+$Comp
+L R_Small R?
+U 1 1 5A2B7511
+P 6000 2350
+AR Path="/5A2AF2A6/5A2B8CFF/5A2B7511" Ref="R?"  Part="1"
+AR Path="/5A2AF2A6/5A2B8A78/5A2B7511" Ref="R?"  Part="1"
+F 0 "R?" V 5900 2300 50  0000 L CNN
+F 1 "R_Small" V 6100 2250 50  0000 L CNN
+F 2 "" H 6000 2350 50  0001 C CNN
+F 3 "" H 6000 2350 50  0001 C CNN
+	1    6000 2350
+	-1   0    0    1
+$EndComp
+$Comp
+L R_Small R?
+U 1 1 5A2B7616
+P 6000 2650
+AR Path="/5A2AF2A6/5A2B8CFF/5A2B7616" Ref="R?"  Part="1"
+AR Path="/5A2AF2A6/5A2B8A78/5A2B7616" Ref="R?"  Part="1"
+F 0 "R?" V 5900 2600 50  0000 L CNN
+F 1 "R_Small" V 6100 2550 50  0000 L CNN
+F 2 "" H 6000 2650 50  0001 C CNN
+F 3 "" H 6000 2650 50  0001 C CNN
+	1    6000 2650
+	-1   0    0    1
+$EndComp
+$Comp
+L GNDPWR #PWR?
+U 1 1 5A2B7666
+P 6000 2950
+AR Path="/5A2AF2A6/5A2B8CFF/5A2B7666" Ref="#PWR?"  Part="1"
+AR Path="/5A2AF2A6/5A2B8A78/5A2B7666" Ref="#PWR?"  Part="1"
+F 0 "#PWR?" H 6000 2750 50  0001 C CNN
+F 1 "GNDPWR" H 6000 2800 50  0000 C CNN
+F 2 "" H 6000 2900 50  0001 C CNN
+F 3 "" H 6000 2900 50  0001 C CNN
+	1    6000 2950
+	1    0    0    -1
+$EndComp
 $EndSCHEMATC
