File: MCU.sch (KiCad schematic (older format))
At the start: 0 parts

Commit message: Moved OpAmp to Chopper.sch
Parts:
- added D?: LED, symbol LED
- added J?: USB_OTG, symbol USB_OTG
- added J? (x2): Conn_01x04, symbol Conn_01x04
- added J?: Conn_ARM_JTAG_SWD_20, symbol Conn_ARM_JTAG_SWD_20
- added R?: R_Small, symbol R_Small
Connections:
- new net GND: J?.10 (GND), J?.12 (GND), J?.14 (GND), J?.16 (GND), J?.18 (GND), J?.20 (GND), J?.4 (GND), J?.6 (GND), J?.8 (GND)
Changed lines of the file:
@@
 Comment4 ""
 $EndDescr
+$Comp
+L USB_OTG J?
+U 1 1 5A27072B
+P 1750 2100
+F 0 "J?" H 1550 2550 50  0000 L CNN
+F 1 "USB_OTG" H 1550 2450 50  0000 L CNN
+F 2 "" H 1900 2050 50  0001 C CNN
+F 3 "" H 1900 2050 50  0001 C CNN
+	1    1750 2100
+	1    0    0    -1
+$EndComp
+$Comp
+L Conn_01x04 J?
+U 1 1 5A270958
+P 9300 5650
+F 0 "J?" H 9300 5850 50  0000 C CNN
+F 1 "Conn_01x04" H 9300 5350 50  0000 C CNN
+F 2 "" H 9300 5650 50  0001 C CNN
+F 3 "" H 9300 5650 50  0001 C CNN
+	1    9300 5650
+	1    0    0    -1
+$EndComp
+$Comp
+L Conn_01x04 J?
+U 1 1 5A27098D
+P 10350 5650
+F 0 "J?" H 10350 5850 50  0000 C CNN
+F 1 "Conn_01x04" H 10350 5350 50  0000 C CNN
+F 2 "" H 10350 5650 50  0001 C CNN
+F 3 "" H 10350 5650 50  0001 C CNN
+	1    10350 5650
+	1    0    0    -1
+$EndComp
+$Comp
+L Conn_ARM_JTAG_SWD_20 J?
+U 1 1 5A2709F3
+P 2050 5700
+F 0 "J?" H 1850 6550 50  0000 R CNN
+F 1 "Conn_ARM_JTAG_SWD_20" H 1850 6450 50  0000 R BNN
+F 2 "" H 2500 4650 50  0001 L TNN
+F 3 "" V 1700 4450 50  0001 C CNN
+	1    2050 5700
+	1    0    0    -1
+$EndComp
+$Comp
+L LED D?
+U 1 1 5A270F2A
+P 9900 1850
+F 0 "D?" H 9900 1950 50  0000 C CNN
+F 1 "LED" H 9900 1750 50  0000 C CNN
+F 2 "" H 9900 1850 50  0001 C CNN
+F 3 "" H 9900 1850 50  0001 C CNN
+	1    9900 1850
+	1    0    0    -1
+$EndComp
+$Comp
+L GNDD #PWR?
+U 1 1 5A270F4F
+P 9850 2150
+F 0 "#PWR?" H 9850 1900 50  0001 C CNN
+F 1 "GNDD" H 9850 2025 50  0000 C CNN
+F 2 "" H 9850 2150 50  0001 C CNN
+F 3 "" H 9850 2150 50  0001 C CNN
+	1    9850 2150
+	1    0    0    -1
+$EndComp
+$Comp
+L +3.3V #PWR?
+U 1 1 5A270F6D
+P 4850 1900
+F 0 "#PWR?" H 4850 1750 50  0001 C CNN
+F 1 "+3.3V" H 4850 2040 50  0000 C CNN
+F 2 "" H 4850 1900 50  0001 C CNN
+F 3 "" H 4850 1900 50  0001 C CNN
+	1    4850 1900
+	1    0    0    -1
+$EndComp
+$Comp
+L R_Small R?
+U 1 1 5A270F90
+P 10150 1700
+F 0 "R?" H 10180 1720 50  0000 L CNN
+F 1 "R_Small" H 10180 1660 50  0000 L CNN
+F 2 "" H 10150 1700 50  0001 C CNN
+F 3 "" H 10150 1700 50  0001 C CNN
+	1    10150 1700
+	1    0    0    -1
+$EndComp
 $EndSCHEMATC
