File: Power.sch (KiCad schematic (older format))
At the start: 0 parts

Commit message: Added Chopper.sch
Parts:
- added C? (x2): C_Small, symbol C_Small
- added D? (x2): LED, symbol LED
- added J?: Screw_Terminal_01x02, symbol Screw_Terminal_01x02
- added Q?: Q_NMOS_GDS, symbol Q_NMOS_GDS
- added R? (x5): R_Small, symbol R_Small
- added U?: AP2127N-3.3, TO_SOT_Packages_SMD:SOT-23, symbol AP2127N-3.3
- added U? (x2): LM358, symbol LM358
Connections:
- net labels added: +3.3V, +5V, GNDPWR, current_desired, current_measured, current_scaled
- wire segments 0 -> 16

Commit message: Moved OpAmp to Chopper.sch
Parts:
- removed Q?: Q_NMOS_GDS, symbol Q_NMOS_GDS
- removed R? (x3): R_Small, symbol R_Small
- removed U? (x2): LM358, symbol LM358
Connections:
- net labels removed: current_desired, current_measured, current_scaled
- wire segments 16 -> 7
Other:
- note added: "add 5V LDO\nand Cs for filtering"
- moved on the sheet: J?
Changed lines of the file:
@@
 L +5V #PWR?
 U 1 1 5A2AFFA3
-P 2450 2350
-F 0 "#PWR?" H 2450 2200 50  0001 C CNN
-F 1 "+5V" H 2450 2490 50  0000 C CNN
-F 2 "" H 2450 2350 50  0001 C CNN
-F 3 "" H 2450 2350 50  0001 C CNN
-	1    2450 2350
+P 1850 2300
+F 0 "#PWR?" H 1850 2150 50  0001 C CNN
+F 1 "+5V" H 1850 2440 50  0000 C CNN
+F 2 "" H 1850 2300 50  0001 C CNN
+F 3 "" H 1850 2300 50  0001 C CNN
+	1    1850 2300
 	1    0    0    -1
 $EndComp
@@
 L GNDPWR #PWR?
 U 1 1 5A2AFFB7
-P 2450 2450
-F 0 "#PWR?" H 2450 2250 50  0001 C CNN
-F 1 "GNDPWR" H 2450 2300 50  0000 C CNN
-F 2 "" H 2450 2400 50  0001 C CNN
-F 3 "" H 2450 2400 50  0001 C CNN
-	1    2450 2450
+P 1850 2400
+F 0 "#PWR?" H 1850 2200 50  0001 C CNN
+F 1 "GNDPWR" H 1850 2250 50  0000 C CNN
+F 2 "" H 1850 2350 50  0001 C CNN
+F 3 "" H 1850 2350 50  0001 C CNN
+	1    1850 2400
 	1    0    0    -1
 $EndComp
@@
 L Screw_Terminal_01x02 J?
 U 1 1 5A2AFFCB
-P 2250 2350
-F 0 "J?" H 2250 2450 50  0000 C CNN
-F 1 "Screw_Terminal_01x02" V 2350 2300 50  0001 C CNN
-F 2 "" H 2250 2350 50  0001 C CNN
-F 3 "" H 2250 2350 50  0001 C CNN
-	1    2250 2350
+P 1650 2300
+F 0 "J?" H 1650 2400 50  0000 C CNN
+F 1 "Screw_Terminal_01x02" V 1750 2250 50  0001 C CNN
+F 2 "" H 1650 2300 50  0001 C CNN
+F 3 "" H 1650 2300 50  0001 C CNN
+	1    1650 2300
 	-1   0    0    -1
 $EndComp
@@
 $EndComp
 Wire Wire Line
-	3150 2550 3750 2550
-Wire Wire Line
-	3750 2550 4300 2550
+	3150 2550 4300 2550
 Connection ~ 3150 2250
 Wire Wire Line
@@
 	3150 2300 3150 2250
 Wire Wire Line
-	4050 2250 4300 2250
-Wire Wire Line
-	4300 2250 4550 2250
+	4050 2250 4550 2250
 Connection ~ 3750 2550
 $Comp
@@
 $EndComp
 Wire Wire Line
-	3450 2250 3150 2250
-Wire Wire Line
-	3150 2250 3000 2250
-$Comp
-L Q_NMOS_GDS Q?
-U 1 1 5A2B4511
-P 7650 3800
-F 0 "Q?" H 7850 3850 50  0000 L CNN
-F 1 "Q_NMOS_GDS" H 7850 3750 50  0000 L CNN
-F 2 "" H 7850 3900 50  0001 C CNN
-F 3 "" H 7650 3800 50  0001 C CNN
-	1    7650 3800
-	1    0    0    -1
-$EndComp
-$Comp
-L LM358 U?
-U 1 1 5A2B487D
-P 6650 2000
-F 0 "U?" H 6650 2200 50  0000 L CNN
-F 1 "LM358" H 6650 1800 50  0000 L CNN
-F 2 "" H 6650 2000 50  0001 C CNN
-F 3 "" H 6650 2000 50  0001 C CNN
-	1    6650 2000
-	1    0    0    -1
-$EndComp
-$Comp
-L LM358 U?
-U 2 1 5A2B48DE
-P 6600 3800
-F 0 "U?" H 6600 4000 50  0000 L CNN
-F 1 "LM358" H 6600 3600 50  0000 L CNN
-F 2 "" H 6600 3800 50  0001 C CNN
-F 3 "" H 6600 3800 50  0001 C CNN
-	2    6600 3800
-	1    0    0    -1
-$EndComp
-$Comp
-L +5V #PWR?
-U 1 1 5A2B4ABD
-P 6500 3500
-F 0 "#PWR?" H 6500 3350 50  0001 C CNN
-F 1 "+5V" H 6500 3640 50  0000 C CNN
-F 2 "" H 6500 3500 50  0001 C CNN
-F 3 "" H 6500 3500 50  0001 C CNN
-	1    6500 3500
-	1    0    0    -1
-$EndComp
-$Comp
-L +5V #PWR?
-U 1 1 5A2B4B1F
-P 6550 1700
-F 0 "#PWR?" H 6550 1550 50  0001 C CNN
-F 1 "+5V" H 6550 1840 50  0000 C CNN
-F 2 "" H 6550 1700 50  0001 C CNN
-F 3 "" H 6550 1700 50  0001 C CNN
-	1    6550 1700
-	1    0    0    -1
-$EndComp
-$Comp
-L GNDPWR #PWR?
-U 1 1 5A2B4F34
-P 6550 2300
-F 0 "#PWR?" H 6550 2100 50  0001 C CNN
-F 1 "GNDPWR" H 6550 2150 50  0000 C CNN
-F 2 "" H 6550 2250 50  0001 C CNN
-F 3 "" H 6550 2250 50  0001 C CNN
-	1    6550 2300
-	1    0    0    -1
-$EndComp
-$Comp
-L GNDPWR #PWR?
-U 1 1 5A2B4F6B
-P 6500 4100
-F 0 "#PWR?" H 6500 3900 50  0001 C CNN
-F 1 "GNDPWR" H 6500 3950 50  0000 C CNN
-F 2 "" H 6500 4050 50  0001 C CNN
-F 3 "" H 6500 4050 50  0001 C CNN
-	1    6500 4100
-	1    0    0    -1
-$EndComp
-$Comp
-L R_Small R?
-U 1 1 5A2B531C
-P 7200 3800
-F 0 "R?" V 7100 3750 50  0000 L CNN
-F 1 "R_Small" V 7300 3700 50  0000 L CNN
-F 2 "" H 7200 3800 50  0001 C CNN
-F 3 "" H 7200 3800 50  0001 C CNN
-	1    7200 3800
-	0    1    1    0
-$EndComp
-Wire Wire Line
-	7300 3800 7450 3800
-Wire Wire Line
-	7100 3800 6900 3800
-$Comp
-L GNDPWR #PWR?
-U 1 1 5A2B5A80
-P 7750 4000
-F 0 "#PWR?" H 7750 3800 50  0001 C CNN
-F 1 "GNDPWR" H 7750 3850 50  0000 C CNN
-F 2 "" H 7750 3950 50  0001 C CNN
-F 3 "" H 7750 3950 50  0001 C CNN
-	1    7750 4000
-	1    0    0    -1
-$EndComp
-Wire Wire Line
-	6300 3900 5900 3900
-Wire Wire Line
-	6300 3700 5900 3700
-Text GLabel 5900 3900 0    60   Input ~ 0
-current_scaled
-Text GLabel 5900 3700 0    60   Input ~ 0
-current_desired
-Text GLabel 8000 2000 0    60   Output ~ 0
-current_scaled
-Wire Wire Line
-	7300 2000 6950 2000
-Wire Wire Line
-	6350 1900 5950 1900
-Text GLabel 5950 1900 0    60   Input ~ 0
-current_measured
-$Comp
-L R_Small R?
-U 1 1 5A2B7511
-P 6000 2350
-F 0 "R?" V 5900 2300 50  0000 L CNN
-F 1 "R_Small" V 6100 2250 50  0000 L CNN
-F 2 "" H 6000 2350 50  0001 C CNN
-F 3 "" H 6000 2350 50  0001 C CNN
-	1    6000 2350
-	-1   0    0    1
-$EndComp
-$Comp
-L R_Small R?
-U 1 1 5A2B7616
-P 6000 2650
-F 0 "R?" V 5900 2600 50  0000 L CNN
-F 1 "R_Small" V 6100 2550 50  0000 L CNN
-F 2 "" H 6000 2650 50  0001 C CNN
-F 3 "" H 6000 2650 50  0001 C CNN
-	1    6000 2650
-	-1   0    0    1
-$EndComp
-$Comp
-L GNDPWR #PWR?
-U 1 1 5A2B7666
-P 6000 2950
-F 0 "#PWR?" H 6000 2750 50  0001 C CNN
-F 1 "GNDPWR" H 6000 2800 50  0000 C CNN
-F 2 "" H 6000 2900 50  0001 C CNN
-F 3 "" H 6000 2900 50  0001 C CNN
-	1    6000 2950
-	1    0    0    -1
-$EndComp
+	3000 2250 3450 2250
 $Sheet
 S 3800 4950 1750 1250
@@
 F1 "Chopper.sch" 60
 $EndSheet
+Text Notes 2100 2400 0    60   ~ 0
+add 5V LDO\nand Cs for filtering
 $EndSCHEMATC
